File: hardware/art-net.kicad_sch (KiCad schematic)
At the start: 31 parts, among them J2 RJ45_Hanrun_HR911105A_Horizon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, U2 D3V3XA4B10LP, U3 LAN8720A

Commit message: fixing issues, adding parts
Parts:
- U2: LCSC (none) -> C1980462
- U3: LCSC (none) -> C45223
Changed lines of the file:
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@@
+			)
+		)
+		(property "LCSC" "C1980462"
+			(at 119.38 93.98 0)
+			(effects
+				(font
+					(size 1.27 1.27)
+				)
+				(hide yes)
 			)
 		)
@@
 			(at 177.8 87.63 0)
 			(effects
+				(font
+					(size 1.27 1.27)
+				)
+				(hide yes)
+			)
+		)
+		(property "LCSC" "C45223"
+			(at 177.8 87.63 0)
+			(effects
