File: hardware/ctrl.kicad_sch (KiCad schematic)
At the start: 18 parts, among them J1 Conn_01x06, Q1 BC817W, Q2 BC817W, U1 ESP32-WROOM-32E, U9 ESP32-C3-WROOM-02

Commit message: fixing issues, adding parts
Parts:
- added J3: USB_C_Receptacle_USB2.0_16P, Connector_USB:USB_C_Receptacle_HCTL_HC-TYPE-C-16P-01A, symbol Connector:USB_C_Receptacle_USB2.0_16P
- added R41, R42: 5k1, Resistor_SMD:R_0603_1608Metric, symbol Device:R
- Q1, Q2: LCSC (none) -> C75566
- U1: LCSC (none) -> C529577
- U9: LCSC (none) -> C2934560
Connections:
- net GND: now also J3.A1 (GND), J3.A12 (GND), J3.B1 (GND), J3.B12 (GND), R41.2, R42.2
- net I2C_~{INT}: now also U9.3 (IO4)
- net TEMP_MON: now also U9.18 (IO0)
- net USB+: now also J3.A6 (D+), J3.B6 (D+)
- net USB-: now also J3.A7 (D-), J3.B7 (D-)
- net VCC_MON: now also U9.17 (IO1)
- net BOOT: now reaches U9.8 (IO9)
- new net: J3.A5 (CC1), R42.1
- new net: J3.A4 (VBUS), J3.A9 (VBUS), J3.B4 (VBUS), J3.B9 (VBUS)
- new net: J3.B5 (CC2), R41.1
- no-connect marks 0 -> 4
