File: hardware/dmx512.kicad_sch (KiCad schematic)
At the start: 18 parts, among them J16 Conn_01x06, J17 Conn_01x06, SW1 SW_DIP_x10, U4 MCP23017T-E/SS, U5 CA-IS3092W

Commit message: fixing issues, adding parts
Parts:
- J16, J17: LCSC (none) -> C274409
Changed lines of the file:
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@@
+			)
+		)
+		(property "LCSC" "C274409"
+			(at 38.1 78.74 0)
+			(effects
+				(font
+					(size 1.27 1.27)
+				)
+				(hide yes)
 			)
 		)
@@
 			(at 38.1 53.34 0)
 			(effects
+				(font
+					(size 1.27 1.27)
+				)
+				(hide yes)
+			)
+		)
+		(property "LCSC" "C274409"
+			(at 38.1 53.34 0)
+			(effects
