File: hardware/emf_beacon.kicad_pcb (KiCad board)
At the start: 2 copper layers, 100 x 100 mm, 146 parts, among them J1 Conn_01x06, J10 Conn_01x02, J11 Conn_01x02, J12 Conn_01x02, J13 Conn_01x02, J14 Conn_01x02, J15 Conn_01x02, J16 Conn_01x06, J17 Conn_01x06, J2 RJ45_Hanrun_HR911105A_Horizon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, J5 Conn_01x02, J6 Conn_01x02, J7 Conn_01x02, J8 Conn_01x02, J9 Conn_01x02, Q1 BC817W, Q10 AO3400A, Q11 AO3400A, Q12 AO3400A, Q13 AO3401A, Q14 BC817W, Q2 BC817W, Q3 AO3400A, Q4 AO3400A, Q5 AO3400A, Q6 AO3400A, Q7 AO3400A, Q8 AO3400A, Q9 AO3400A, SW1 SW_DIP_x10, U1 ESP32-WROOM-32E, U2 D3V3XA4B10LP, U3 LAN8720A, U4 MCP23017T-E/SS, U5 CA-IS3092W, U6 PCA9685PW, U7 ZTP7193MA, U8 ZTP7193MA, U9 ESP32-C3-WROOM-02

Commit message: fixing issues, adding parts
Parts:
- removed C28, C34: 47uF, Capacitor_SMD:C_1210_3225Metric
- removed C30: 100nF, Capacitor_SMD:C_0603_1608Metric
- removed C32: 1uF, Capacitor_SMD:C_0603_1608Metric
- removed L1: IHLP2525CZER100M01, Inductor_SMD:L_Vishay_IHLP-2525
- removed R43: 100k, Resistor_SMD:R_0603_1608Metric
- removed R47: 33k, Resistor_SMD:R_0603_1608Metric
- removed R49: 36k, Resistor_SMD:R_0603_1608Metric
- removed R50: 4k3, Resistor_SMD:R_0603_1608Metric
- removed TP5, TP6: TestPoint, TestPoint:TestPoint_Pad_D1.5mm
- removed U7: ZTP7193MA, Package_TO_SOT_SMD:SOT-23-8
- added C37: C, Capacitor_SMD:C_1210_3225Metric, F.Cu at (222.6, 128.4)
- added C38: 470pF, Capacitor_SMD:C_0603_1608Metric, F.Cu at (209.7, 109.2)
- added C39: 1uF, Capacitor_SMD:C_0603_1608Metric, F.Cu at (209.7, 111.7)
- added C40: 22uF, Capacitor_SMD:C_1206_3216Metric, F.Cu at (227.6, 109.6)
- added C41: 22uF, Capacitor_SMD:C_1206_3216Metric, F.Cu at (227.6, 113.0)
- added D3: SS34, Diode_SMD:D_SMA, F.Cu at (215.8, 122.0)
- added D4: SMAJ15A, Diode_SMD:D_SMA, F.Cu at (215.8, 126.5)
- added J3: USB_C_Receptacle_USB2.0_16P, Connector_USB:USB_C_Receptacle_HCTL_HC-TYPE-C-16P-01A, F.Cu at (238.7, 113.4)
- added L3: JSHC1040H-4R7M-G, Inductor_SMD:L_Wuerth_HCI-1040, F.Cu at (218.2, 113.8)
- added R56: 33k, Resistor_SMD:R_0603_1608Metric, F.Cu at (209.7, 114.2)
- added R57: 10k, Resistor_SMD:R_0603_1608Metric, F.Cu at (209.7, 116.7)
- added R58: 200k, Resistor_SMD:R_0603_1608Metric, F.Cu at (209.7, 119.2)
- added R59: 150k, Resistor_SMD:R_0603_1608Metric, F.Cu at (209.7, 121.8)
- added R60: 16k, Resistor_SMD:R_0603_1608Metric, F.Cu at (209.7, 124.3)
- added U10: FP6151XR-G1, Package_SO:HSOP-8-1EP_3.9x4.9mm_P1.27mm_EP2.41x3.1mm, F.Cu at (224.0, 123.1)
- C27: value 1uF -> 100nF 50V
- D2: value ZMM5V6-M -> BZT52C10; footprint Diode_SMD:D_MiniMELF -> Diode_SMD:D_SOD-123; moved to F.Cu
- Q13: value AO3401A -> DMP3013SFV; footprint Package_TO_SOT_SMD:SOT-23 -> Package_SON:Diodes_PowerDI3333-8; moved to F.Cu
- R41: value 91k -> 5k1; moved to F.Cu
- R42: value 10k -> 5k1; moved to F.Cu
- moved R42 107.1 mm to (234.9, 121.8), turned to 0 degrees
- moved R41 105.6 mm to (234.9, 119.3), turned to 0 degrees
- moved D2 74.5 mm to (227.7, 116.3), turned to 0 degrees
- moved Q13 42.0 mm to (228.2, 128.8), turned to 0 degrees
Connections:
- C27 pad 1: VDC -> Net-(J15-Pin_2)
- C29 pad 1: +12V -> VDC
- D2 pad 1: Net-(D2-K) -> VDC
- J15 pad 2: VDC -> Net-(J15-Pin_2)
- Q13 pad 1: Net-(D2-A) -> VDC
- Q13 pad 2: Net-(D2-K) -> VDC
- R41 pad 1: /POWER/VCC_6V5 -> Net-(J3-CC2)
- R41 pad 2: Net-(U7-AAM) -> GND
- R42 pad 1: Net-(U7-AAM) -> Net-(J3-CC1)
- R46 pad 1: +12V -> VDC
- TP1 pad 1: VDC -> Net-(J15-Pin_2)
- U8 pad 2: +12V -> VDC
- U9 pad 17: unconnected-(U9-IO1-Pad17) -> /CTRL/VCC_MON
- U9 pad 18: unconnected-(U9-IO0-Pad18) -> /CTRL/TEMP_MON
- U9 pad 3: unconnected-(U9-IO4-Pad3) -> /CTRL/I2C_~{INT}
- U9 pad 8: unconnected-(U9-IO9-Pad8) -> /CTRL/BOOT
Routing:
- added copper zone on B.Cu, net VDC
- removed copper zone on B.Cu, net +12V
- removed copper zone on B.Cu, net /POWER/SW_6V5
