File: hardware/leds.kicad_sch (KiCad schematic)
At the start: 36 parts, among them J10 Conn_01x02, J11 Conn_01x02, J12 Conn_01x02, J13 Conn_01x02, J14 Conn_01x02, J5 Conn_01x02, J6 Conn_01x02, J7 Conn_01x02, J8 Conn_01x02, J9 Conn_01x02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

Commit message: fixing issues, adding parts
Other:
- note added: "Snubbers? 10R 0402 & 10nF 0402 across Vds"
Changed lines of the file:
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@@
+		)
+	)
+	(text "Snubbers?\n10R 0402 & 10nF 0402 across Vds"
+		(exclude_from_sim no)
+		(at 143.764 169.926 0)
+		(effects
+			(font
+				(size 2.54 2.54)
+				(color 255 0 0 1)
+			)
 		)
 	)
